File: train_horn.kicad_pcb (KiCad board)
At the start: 2 copper layers, 33 x 100 mm, 104 parts, among them J1 USB_OTG, J2 PROG, Q1 2N7002, SW1 PLAY, U1 MIC7221, U2 MCP73831, U3 TPS78233DDCR, U4 MSP430FR2000_TSSOP, U5 TPA6211A1

Commit message: update LED ref to reflect ref on schematic
Parts:
- D1: value RED -> BLUE
- D2: value LED -> RED
- D3: value PLAYING -> GREEN
Changed lines of the file:
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@@
       (effects (font (size 1 1) (thickness 0.15)))
     )
-    (fp_text value RED (at 0 1.3) (layer F.Fab)
+    (fp_text value BLUE (at 0 1.3) (layer F.Fab)
       (effects (font (size 0.5 0.5) (thickness 0.125)))
     )
@@
       (effects (font (size 1 1) (thickness 0.15)))
     )
-    (fp_text value LED (at 0 1.3) (layer F.Fab)
+    (fp_text value RED (at 0 1.3) (layer F.Fab)
       (effects (font (size 0.5 0.5) (thickness 0.125)))
     )
@@
       (effects (font (size 1 1) (thickness 0.15)))
     )
-    (fp_text value PLAYING (at 0 1.3) (layer F.Fab)
+    (fp_text value GREEN (at 0 1.3) (layer F.Fab)
       (effects (font (size 0.5 0.5) (thickness 0.125)))
     )
